File: hardware/ecp5_mainboard/fpga_io.sch (KiCad schematic (older format))
At the start: 76 parts, among them J10 UART, J11 FLASH, J12 JTAG, J5 EXT0, J6 EXT1, J7 EXT2, J9 PMOD_01, Q9 BSH111BKR, SW6 SW_Push, U15 ECP5UM5G_85_CABGA756, U26 XL_XO_LVDS, U27 W25Q

Commit message: U27 changed to upstream KiCAD symbol
Parts:
- removed U27: W25Q, Package_SO:SO-8_5.3x6.2mm_P1.27mm, symbol ecp5_mainboard-rescue:W25Q-pkl_memory
- added U27: W25Q128JVS, Package_SO:SOIC-8_5.23x5.23mm_P1.27mm, symbol Memory_Flash:W25Q128JVS
Connections:
- wire segments 888 -> 891
Other:
- moved on the sheet: C251
Changed lines of the file:
@@
 EESchema Schematic File Version 4
 LIBS:ecp5_mainboard-cache
-EELAYER 29 0
+EELAYER 30 0
 EELAYER END
 $Descr A2 23386 16535
@@
 Text Label 20750 8300 0    50   ~ 0
 ~INIT
-$Comp
-L ecp5_mainboard-rescue:W25Q-pkl_memory U27
-U 1 1 60E46888
-P 20600 9650
-AR Path="/60E46888" Ref="U27"  Part="1"
-AR Path="/61FAF948/60E46888" Ref="U27"  Part="1"
-F 0 "U27" H 20600 10075 50  0000 C CNN
-F 1 "W25Q" H 20600 9984 50  0000 C CNN
-F 2 "Package_SO:SO-8_5.3x6.2mm_P1.27mm" H 20600 9650 50  0001 C CNN
-F 3 "" H 20600 9650 50  0001 C CNN
-	1    20600 9650
-	1    0    0    -1
-$EndComp
-Wire Wire Line
-	20000 9450 18900 9450
-Wire Wire Line
-	20000 9550 19200 9550
 Wire Wire Line
-	20000 9650 19500 9650
+	20000 9550 19500 9550
 Wire Wire Line
-	20000 9750 19600 9750
+	20000 9650 19600 9650
 Wire Wire Line
 	20000 9850 19700 9850
@@
 $EndComp
 Wire Wire Line
-	19500 9400 19500 9650
+	19500 9400 19500 9550
 Connection ~ 19500 9650
 Wire Wire Line
 	19500 9650 18150 9650
 Wire Wire Line
-	19600 9400 19600 9750
+	19600 9400 19600 9650
 Connection ~ 19600 9750
 Wire Wire Line
@@
 Wire Wire Line
 	19200 9300 19200 9550
-Connection ~ 19200 9550
 Wire Wire Line
 	19200 9550 18700 9550
 Wire Wire Line
 	18900 9300 18900 9450
-Connection ~ 18900 9450
 Wire Wire Line
 	18900 9450 18800 9450
@@
 Connection ~ 18900 8900
 $Comp
-L power:+3V3 #PWR0242
-U 1 1 61D7915B
-P 21300 9300
-F 0 "#PWR0242" H 21300 9150 50  0001 C CNN
-F 1 "+3V3" H 21315 9473 50  0000 C CNN
-F 2 "" H 21300 9300 50  0001 C CNN
-F 3 "" H 21300 9300 50  0001 C CNN
-	1    21300 9300
-	1    0    0    -1
-$EndComp
-Wire Wire Line
-	21300 9300 21300 9450
-Wire Wire Line
-	21300 9450 21200 9450
-$Comp
 L power:GND #PWR0243
 U 1 1 61E38305
-P 21300 10100
-F 0 "#PWR0243" H 21300 9850 50  0001 C CNN
-F 1 "GND" H 21305 9927 50  0000 C CNN
-F 2 "" H 21300 10100 50  0001 C CNN
-F 3 "" H 21300 10100 50  0001 C CNN
-	1    21300 10100
+P 21600 10300
+F 0 "#PWR0243" H 21600 10050 50  0001 C CNN
+F 1 "GND" H 21605 10127 50  0000 C CNN
+F 2 "" H 21600 10300 50  0001 C CNN
+F 3 "" H 21600 10300 50  0001 C CNN
+	1    21600 10300
 	1    0    0    -1
 $EndComp
 Wire Wire Line
-	21300 10100 21300 9950
-Wire Wire Line
-	21300 9950 21200 9950
+	21600 10300 21600 10150
 $Comp
 L Device:C_Small C251
 U 1 1 61EF7C86
-P 21300 9700
-F 0 "C251" H 21392 9746 50  0000 L CNN
-F 1 "470n" H 21392 9655 50  0000 L CNN
-F 2 "Capacitor_SMD:C_0402_1005Metric" H 21300 9700 50  0001 C CNN
-F 3 "~" H 21300 9700 50  0001 C CNN
-	1    21300 9700
+P 21600 9900
+F 0 "C251" H 21692 9946 50  0000 L CNN
+F 1 "470n" H 21692 9855 50  0000 L CNN
+F 2 "Capacitor_SMD:C_0402_1005Metric" H 21600 9900 50  0001 C CNN
+F 3 "~" H 21600 9900 50  0001 C CNN
+	1    21600 9900
 	1    0    0    -1
 $EndComp
 Wire Wire Line
-	21300 9600 21300 9450
-Connection ~ 21300 9450
-Wire Wire Line
-	21300 9800 21300 9950
-Connection ~ 21300 9950
+	21600 10000 21600 10150
+Connection ~ 21600 10150
 $Comp
 L ECP5UM5G:ECP5UM5G_85_CABGA756 U15
@@
 NoConn ~ 12550 10900
 NoConn ~ 12550 11100
+$Comp
+L Memory_Flash:W25Q128JVS U27
+U 1 1 5DFB9E60
+P 20500 9750
+F 0 "U27" H 20850 10100 50  0000 C CNN
+F 1 "W25Q128JVS" H 20200 10100 50  0000 C CNN
+F 2 "Package_SO:SOIC-8_5.23x5.23mm_P1.27mm" H 20500 9750 50  0001 C CNN
+F 3 "http://www.winbond.com/resource-files/w25q128jv_dtr%20revc%2003272018%20plus.pdf" H 20500 9750 50  0001 C CNN
+	1    20500 9750
+	-1   0    0    -1
+$EndComp
+Connection ~ 19500 9550
+Wire Wire Line
+	19500 9550 19500 9650
+Connection ~ 19600 9650
+Wire Wire Line
+	19600 9650 19600 9750
+$Comp
+L power:+3V3 #PWR0242
+U 1 1 61D7915B
+P 20500 9250
+F 0 "#PWR0242" H 20500 9100 50  0001 C CNN
+F 1 "+3V3" H 20515 9423 50  0000 C CNN
+F 2 "" H 20500 9250 50  0001 C CNN
+F 3 "" H 20500 9250 50  0001 C CNN
+	1    20500 9250
+	1    0    0    -1
+$EndComp
+Wire Wire Line
+	20500 9350 20500 9300
+Wire Wire Line
+	20500 10150 21600 10150
+Text Label 21100 9650 0    50   ~ 0
+FLASH_~CS
+Text Label 21100 9850 0    50   ~ 0
+FLASH_CLK
+Wire Wire Line
+	21000 9650 21100 9650
+Wire Wire Line
+	21000 9850 21100 9850
+Wire Wire Line
+	21600 9800 21600 9300
+Wire Wire Line
+	21600 9300 20500 9300
+Connection ~ 20500 9300
+Wire Wire Line
+	20500 9300 20500 9250
 $EndSCHEMATC

Commit message: Revert "U27 changed to upstream KiCAD symbol"
This reverts commit d96042e48b49db5ee8c05d0d117dc24b07897af7.
Parts:
- removed U27: W25Q128JVS, Package_SO:SOIC-8_5.23x5.23mm_P1.27mm, symbol Memory_Flash:W25Q128JVS
- added U27: W25Q, Package_SO:SO-8_5.3x6.2mm_P1.27mm, symbol ecp5_mainboard-rescue:W25Q-pkl_memory
Connections:
- wire segments 891 -> 888
Other:
- moved on the sheet: C251
Changed lines of the file:
@@
 EESchema Schematic File Version 4
 LIBS:ecp5_mainboard-cache
-EELAYER 30 0
+EELAYER 29 0
 EELAYER END
 $Descr A2 23386 16535
@@
 Text Label 20750 8300 0    50   ~ 0
 ~INIT
+$Comp
+L ecp5_mainboard-rescue:W25Q-pkl_memory U27
+U 1 1 60E46888
+P 20600 9650
+AR Path="/60E46888" Ref="U27"  Part="1"
+AR Path="/61FAF948/60E46888" Ref="U27"  Part="1"
+F 0 "U27" H 20600 10075 50  0000 C CNN
+F 1 "W25Q" H 20600 9984 50  0000 C CNN
+F 2 "Package_SO:SO-8_5.3x6.2mm_P1.27mm" H 20600 9650 50  0001 C CNN
+F 3 "" H 20600 9650 50  0001 C CNN
+	1    20600 9650
+	1    0    0    -1
+$EndComp
+Wire Wire Line
+	20000 9450 18900 9450
+Wire Wire Line
+	20000 9550 19200 9550
 Wire Wire Line
-	20000 9550 19500 9550
+	20000 9650 19500 9650
 Wire Wire Line
-	20000 9650 19600 9650
+	20000 9750 19600 9750
 Wire Wire Line
 	20000 9850 19700 9850
@@
 $EndComp
 Wire Wire Line
-	19500 9400 19500 9550
+	19500 9400 19500 9650
 Connection ~ 19500 9650
 Wire Wire Line
 	19500 9650 18150 9650
 Wire Wire Line
-	19600 9400 19600 9650
+	19600 9400 19600 9750
 Connection ~ 19600 9750
 Wire Wire Line
@@
 Wire Wire Line
 	19200 9300 19200 9550
+Connection ~ 19200 9550
 Wire Wire Line
 	19200 9550 18700 9550
 Wire Wire Line
 	18900 9300 18900 9450
+Connection ~ 18900 9450
 Wire Wire Line
 	18900 9450 18800 9450
@@
 Connection ~ 18900 8900
 $Comp
+L power:+3V3 #PWR0242
+U 1 1 61D7915B
+P 21300 9300
+F 0 "#PWR0242" H 21300 9150 50  0001 C CNN
+F 1 "+3V3" H 21315 9473 50  0000 C CNN
+F 2 "" H 21300 9300 50  0001 C CNN
+F 3 "" H 21300 9300 50  0001 C CNN
+	1    21300 9300
+	1    0    0    -1
+$EndComp
+Wire Wire Line
+	21300 9300 21300 9450
+Wire Wire Line
+	21300 9450 21200 9450
+$Comp
 L power:GND #PWR0243
 U 1 1 61E38305
-P 21600 10300
-F 0 "#PWR0243" H 21600 10050 50  0001 C CNN
-F 1 "GND" H 21605 10127 50  0000 C CNN
-F 2 "" H 21600 10300 50  0001 C CNN
-F 3 "" H 21600 10300 50  0001 C CNN
-	1    21600 10300
+P 21300 10100
+F 0 "#PWR0243" H 21300 9850 50  0001 C CNN
+F 1 "GND" H 21305 9927 50  0000 C CNN
+F 2 "" H 21300 10100 50  0001 C CNN
+F 3 "" H 21300 10100 50  0001 C CNN
+	1    21300 10100
 	1    0    0    -1
 $EndComp
 Wire Wire Line
-	21600 10300 21600 10150
+	21300 10100 21300 9950
+Wire Wire Line
+	21300 9950 21200 9950
 $Comp
 L Device:C_Small C251
 U 1 1 61EF7C86
-P 21600 9900
-F 0 "C251" H 21692 9946 50  0000 L CNN
-F 1 "470n" H 21692 9855 50  0000 L CNN
-F 2 "Capacitor_SMD:C_0402_1005Metric" H 21600 9900 50  0001 C CNN
-F 3 "~" H 21600 9900 50  0001 C CNN
-	1    21600 9900
+P 21300 9700
+F 0 "C251" H 21392 9746 50  0000 L CNN
+F 1 "470n" H 21392 9655 50  0000 L CNN
+F 2 "Capacitor_SMD:C_0402_1005Metric" H 21300 9700 50  0001 C CNN
+F 3 "~" H 21300 9700 50  0001 C CNN
+	1    21300 9700
 	1    0    0    -1
 $EndComp
 Wire Wire Line
-	21600 10000 21600 10150
-Connection ~ 21600 10150
+	21300 9600 21300 9450
+Connection ~ 21300 9450
+Wire Wire Line
+	21300 9800 21300 9950
+Connection ~ 21300 9950
 $Comp
 L ECP5UM5G:ECP5UM5G_85_CABGA756 U15
@@
 NoConn ~ 12550 10900
 NoConn ~ 12550 11100
-$Comp
-L Memory_Flash:W25Q128JVS U27
-U 1 1 5DFB9E60
-P 20500 9750
-F 0 "U27" H 20850 10100 50  0000 C CNN
-F 1 "W25Q128JVS" H 20200 10100 50  0000 C CNN
-F 2 "Package_SO:SOIC-8_5.23x5.23mm_P1.27mm" H 20500 9750 50  0001 C CNN
-F 3 "http://www.winbond.com/resource-files/w25q128jv_dtr%20revc%2003272018%20plus.pdf" H 20500 9750 50  0001 C CNN
-	1    20500 9750
-	-1   0    0    -1
-$EndComp
-Connection ~ 19500 9550
-Wire Wire Line
-	19500 9550 19500 9650
-Connection ~ 19600 9650
-Wire Wire Line
-	19600 9650 19600 9750
-$Comp
-L power:+3V3 #PWR0242
-U 1 1 61D7915B
-P 20500 9250
-F 0 "#PWR0242" H 20500 9100 50  0001 C CNN
-F 1 "+3V3" H 20515 9423 50  0000 C CNN
-F 2 "" H 20500 9250 50  0001 C CNN
-F 3 "" H 20500 9250 50  0001 C CNN
-	1    20500 9250
-	1    0    0    -1
-$EndComp
-Wire Wire Line
-	20500 9350 20500 9300
-Wire Wire Line
-	20500 10150 21600 10150
-Text Label 21100 9650 0    50   ~ 0
-FLASH_~CS
-Text Label 21100 9850 0    50   ~ 0
-FLASH_CLK
-Wire Wire Line
-	21000 9650 21100 9650
-Wire Wire Line
-	21000 9850 21100 9850
-Wire Wire Line
-	21600 9800 21600 9300
-Wire Wire Line
-	21600 9300 20500 9300
-Connection ~ 20500 9300
-Wire Wire Line
-	20500 9300 20500 9250
 $EndSCHEMATC
