File: hardware/ecp5_mainboard/fpga_io.sch (KiCad schematic (older format))
At the start: 76 parts, among them J10 UART, J11 FLASH, J12 JTAG, J5 EXT0, J6 EXT1, J7 EXT2, J9 PMOD_01, Q9 BSH111BKR, SW6 SW_Push, U15 ECP5UM5G_85_CABGA756, U26 XL_XO_LVDS, U27 W25Q

Commit message: U26 symbol changed to upstream
Parts:
- removed U26: XL_XO_LVDS, Custom Parts:OSC_IDT_XU_5x3.2mm, symbol eco_glue:XL_XO_LVDS
- added U26: XUL535100.000JS6I8, Oscillator:Oscillator_SMD_IDT_JS6-6_5.0x3.2mm_P1.27mm, symbol Oscillator:XUX53
Connections:
- wire segments 888 -> 887
- no-connect marks 64 -> 63
Changed lines of the file:
@@
 EESchema Schematic File Version 4
 LIBS:ecp5_mainboard-cache
-EELAYER 29 0
+EELAYER 30 0
 EELAYER END
 $Descr A2 23386 16535
@@
 	15050 6500 15400 6500
 $Comp
-L eco_glue:XL_XO_LVDS U26
-U 1 1 6249D25D
-P 20150 1400
-F 0 "U26" H 20150 1865 50  0000 C CNN
-F 1 "XL_XO_LVDS" H 20150 1774 50  0000 C CNN
-F 2 "Custom Parts:OSC_IDT_XU_5x3.2mm" H 20150 1400 50  0001 C CNN
-F 3 "" H 20150 1400 50  0001 C CNN
-	1    20150 1400
-	1    0    0    -1
-$EndComp
-$Comp
 L power:GND #PWR0234
 U 1 1 6249D389
-P 19250 1750
-F 0 "#PWR0234" H 19250 1500 50  0001 C CNN
-F 1 "GND" H 19255 1577 50  0000 C CNN
-F 2 "" H 19250 1750 50  0001 C CNN
-F 3 "" H 19250 1750 50  0001 C CNN
-	1    19250 1750
+P 20850 1950
+F 0 "#PWR0234" H 20850 1700 50  0001 C CNN
+F 1 "GND" H 20855 1777 50  0000 C CNN
+F 2 "" H 20850 1950 50  0001 C CNN
+F 3 "" H 20850 1950 50  0001 C CNN
+	1    20850 1950
 	1    0    0    -1
 $EndComp
-Wire Wire Line
-	19250 1750 19250 1600
-Wire Wire Line
-	19250 1600 19450 1600
-NoConn ~ 19450 1400
-NoConn ~ 19450 1200
+NoConn ~ 20450 1650
 $Comp
 L power:+3V3 #PWR0240
@@
 	0    1    1    0
 $EndComp
-Text Label 21800 1400 2    50   ~ 0
-CLK100-
-Wire Wire Line
-	21800 1400 20850 1400
-Text Label 21800 1600 2    50   ~ 0
-CLK100+
-Wire Wire Line
-	21800 1600 20850 1600
 Text GLabel 15050 4800 0    50   BiDi ~ 0
 CLK_SDA
@@
 NoConn ~ 12550 10900
 NoConn ~ 12550 11100
+$Comp
+L Oscillator:XUX53 U26
+U 1 1 5E0DB69A
+P 20850 1650
+F 0 "U26" H 20600 1900 50  0000 C CNN
+F 1 "XUL535100.000JS6I8 " H 21300 1900 50  0000 C CNN
+F 2 "Oscillator:Oscillator_SMD_IDT_JS6-6_5.0x3.2mm_P1.27mm" H 20900 1300 50  0001 C CNN
+F 3 "https://www.idt.com/document/dst/xu-family-datasheet" H 20450 2350 50  0001 C CNN
+	1    20850 1650
+	1    0    0    -1
+$EndComp
+Wire Wire Line
+	22200 1650 21250 1650
+Text Label 22200 1650 2    50   ~ 0
+CLK100+
+Wire Wire Line
+	22200 1750 21250 1750
+Text Label 22200 1750 2    50   ~ 0
+CLK100-
+Wire Wire Line
+	20850 1200 20850 1350
 $EndSCHEMATC
