File: hardware/ecp5_mainboard/fpga_io.sch (KiCad schematic (older format))
At the start: 76 parts, among them J10 UART, J11 FLASH, J12 JTAG, J5 EXT0, J6 EXT1, J7 EXT2, J9 PMOD_01, Q9 BSH111BKR, SW6 SW_Push, U15 ECP5UM5G_85_CABGA756, U26 XUL535100.000JS6I8, U27 W25Q

Commit message: U27 changed to upstream KiCAD symbol
Parts:
- removed U27: W25Q, Package_SO:SO-8_5.3x6.2mm_P1.27mm, symbol ecp5_mainboard-rescue:W25Q-pkl_memory
- added U27: W25Q128JVS, Package_SO:SOIC-8_5.23x5.23mm_P1.27mm, symbol Memory_Flash:W25Q128JVS
Connections:
- wire segments 887 -> 882
Other:
- moved on the sheet: C251, R88, R89
Changed lines of the file:
@@
 EESchema Schematic File Version 4
-LIBS:ecp5_mainboard-cache
 EELAYER 30 0
 EELAYER END
@@
 ~INIT
 $Comp
-L ecp5_mainboard-rescue:W25Q-pkl_memory U27
-U 1 1 60E46888
-P 20600 9650
-AR Path="/60E46888" Ref="U27"  Part="1"
-AR Path="/61FAF948/60E46888" Ref="U27"  Part="1"
-F 0 "U27" H 20600 10075 50  0000 C CNN
-F 1 "W25Q" H 20600 9984 50  0000 C CNN
-F 2 "Package_SO:SO-8_5.3x6.2mm_P1.27mm" H 20600 9650 50  0001 C CNN
-F 3 "" H 20600 9650 50  0001 C CNN
-	1    20600 9650
-	1    0    0    -1
-$EndComp
-Wire Wire Line
-	20000 9450 18900 9450
-Wire Wire Line
-	20000 9550 19200 9550
-Wire Wire Line
-	20000 9650 19500 9650
-Wire Wire Line
-	20000 9750 19600 9750
-Wire Wire Line
-	20000 9850 19700 9850
-Wire Wire Line
-	20000 9950 19800 9950
-$Comp
 L Device:R_Small R88
 U 1 1 6128A4E3
-P 18900 9200
-F 0 "R88" H 18959 9246 50  0000 L CNN
-F 1 "4.7k" H 18959 9155 50  0000 L CNN
-F 2 "Resistor_SMD:R_0402_1005Metric" H 18900 9200 50  0001 C CNN
-F 3 "~" H 18900 9200 50  0001 C CNN
-	1    18900 9200
+P 21200 9450
+F 0 "R88" H 21259 9496 50  0000 L CNN
+F 1 "4.7k" H 21259 9405 50  0000 L CNN
+F 2 "Resistor_SMD:R_0402_1005Metric" H 21200 9450 50  0001 C CNN
+F 3 "~" H 21200 9450 50  0001 C CNN
+	1    21200 9450
 	1    0    0    -1
 $EndComp
@@
 L Device:R_Small R89
 U 1 1 613418D6
-P 19200 9200
-F 0 "R89" H 19259 9246 50  0000 L CNN
-F 1 "1k" H 19259 9155 50  0000 L CNN
-F 2 "Resistor_SMD:R_0402_1005Metric" H 19200 9200 50  0001 C CNN
-F 3 "~" H 19200 9200 50  0001 C CNN
-	1    19200 9200
+P 21500 9450
+F 0 "R89" H 21559 9496 50  0000 L CNN
+F 1 "1k" H 21559 9405 50  0000 L CNN
+F 2 "Resistor_SMD:R_0402_1005Metric" H 21500 9450 50  0001 C CNN
+F 3 "~" H 21500 9450 50  0001 C CNN
+	1    21500 9450
 	1    0    0    -1
 $EndComp
@@
 $EndComp
 Wire Wire Line
-	19500 9400 19500 9650
-Connection ~ 19500 9650
-Wire Wire Line
-	19500 9650 18150 9650
-Wire Wire Line
-	19600 9400 19600 9750
-Connection ~ 19600 9750
+	19500 9400 19500 9550
 Wire Wire Line
-	19600 9750 18150 9750
+	19600 9400 19600 9650
 Wire Wire Line
 	19700 9400 19700 9850
@@
 	19800 9950 18150 9950
 Wire Wire Line
-	19200 9300 19200 9550
-Connection ~ 19200 9550
-Wire Wire Line
-	19200 9550 18700 9550
-Wire Wire Line
-	18900 9300 18900 9450
-Connection ~ 18900 9450
-Wire Wire Line
-	18900 9450 18800 9450
-Wire Wire Line
-	18900 9100 18900 8900
-Wire Wire Line
 	19800 8900 19800 9000
 Wire Wire Line
@@
 	19700 8900 19800 8900
 Wire Wire Line
-	19200 9100 19200 8900
-Wire Wire Line
-	18900 8900 19200 8900
-Connection ~ 19200 8900
-Wire Wire Line
-	19200 8900 19500 8900
-Wire Wire Line
 	19500 9000 19500 8900
-Connection ~ 19500 8900
 Wire Wire Line
 	19500 8900 19600 8900
@@
 L power:+3V3 #PWR0232
 U 1 1 61BFC583
-P 18900 8800
-F 0 "#PWR0232" H 18900 8650 50  0001 C CNN
-F 1 "+3V3" H 18915 8973 50  0000 C CNN
-F 2 "" H 18900 8800 50  0001 C CNN
-F 3 "" H 18900 8800 50  0001 C CNN
-	1    18900 8800
+P 19600 8800
+F 0 "#PWR0232" H 19600 8650 50  0001 C CNN
+F 1 "+3V3" H 19615 8973 50  0000 C CNN
+F 2 "" H 19600 8800 50  0001 C CNN
+F 3 "" H 19600 8800 50  0001 C CNN
+	1    19600 8800
 	1    0    0    -1
 $EndComp
-Wire Wire Line
-	18900 8800 18900 8900
-Connection ~ 18900 8900
 $Comp
 L power:+3V3 #PWR0242
 U 1 1 61D7915B
-P 21300 9300
-F 0 "#PWR0242" H 21300 9150 50  0001 C CNN
-F 1 "+3V3" H 21315 9473 50  0000 C CNN
-F 2 "" H 21300 9300 50  0001 C CNN
-F 3 "" H 21300 9300 50  0001 C CNN
-	1    21300 9300
+P 22150 9250
+F 0 "#PWR0242" H 22150 9100 50  0001 C CNN
+F 1 "+3V3" H 22165 9423 50  0000 C CNN
+F 2 "" H 22150 9250 50  0001 C CNN
+F 3 "" H 22150 9250 50  0001 C CNN
+	1    22150 9250
 	1    0    0    -1
 $EndComp
-Wire Wire Line
-	21300 9300 21300 9450
-Wire Wire Line
-	21300 9450 21200 9450
 $Comp
 L power:GND #PWR0243
 U 1 1 61E38305
-P 21300 10100
-F 0 "#PWR0243" H 21300 9850 50  0001 C CNN
-F 1 "GND" H 21305 9927 50  0000 C CNN
-F 2 "" H 21300 10100 50  0001 C CNN
-F 3 "" H 21300 10100 50  0001 C CNN
-	1    21300 10100
+P 22150 10150
+F 0 "#PWR0243" H 22150 9900 50  0001 C CNN
+F 1 "GND" H 22155 9977 50  0000 C CNN
+F 2 "" H 22150 10150 50  0001 C CNN
+F 3 "" H 22150 10150 50  0001 C CNN
+	1    22150 10150
 	1    0    0    -1
 $EndComp
-Wire Wire Line
-	21300 10100 21300 9950
-Wire Wire Line
-	21300 9950 21200 9950
 $Comp
 L Device:C_Small C251
 U 1 1 61EF7C86
-P 21300 9700
-F 0 "C251" H 21392 9746 50  0000 L CNN
-F 1 "470n" H 21392 9655 50  0000 L CNN
-F 2 "Capacitor_SMD:C_0402_1005Metric" H 21300 9700 50  0001 C CNN
-F 3 "~" H 21300 9700 50  0001 C CNN
-	1    21300 9700
+P 22150 9700
+F 0 "C251" H 22242 9746 50  0000 L CNN
+F 1 "470n" H 22242 9655 50  0000 L CNN
+F 2 "Capacitor_SMD:C_0402_1005Metric" H 22150 9700 50  0001 C CNN
+F 3 "~" H 22150 9700 50  0001 C CNN
+	1    22150 9700
 	1    0    0    -1
 $EndComp
-Wire Wire Line
-	21300 9600 21300 9450
-Connection ~ 21300 9450
-Wire Wire Line
-	21300 9800 21300 9950
-Connection ~ 21300 9950
 $Comp
 L ECP5UM5G:ECP5UM5G_85_CABGA756 U15
@@
 Wire Wire Line
 	20100 12350 19750 12350
-Text Label 18150 9550 0    50   ~ 0
+Text Label 22000 9850 2    50   ~ 0
 FLASH_CLK
-Text Label 18150 9450 0    50   ~ 0
+Text Label 18150 10350 0    50   ~ 0
 FLASH_~CS
-Text Label 18150 9650 0    50   ~ 0
-FLASH_D0
-Text Label 18150 9750 0    50   ~ 0
-FLASH_D1
 Text Label 18150 9850 0    50   ~ 0
 FLASH_D2
@@
 	19400 10250 19500 10250
 Wire Wire Line
-	19500 10250 19500 9650
-Wire Wire Line
-	19600 9750 19600 10350
-Wire Wire Line
 	19600 10350 19400 10350
 Wire Wire Line
@@
 Wire Wire Line
 	19800 10550 19400 10550
-Wire Wire Line
-	18900 10350 18800 10350
-Wire Wire Line
-	18800 10350 18800 9450
-Connection ~ 18800 9450
-Wire Wire Line
-	18800 9450 18150 9450
-Wire Wire Line
-	18900 10450 18700 10450
-Wire Wire Line
-	18700 10450 18700 9550
-Connection ~ 18700 9550
-Wire Wire Line
-	18700 9550 18150 9550
 $Comp
 L power:GND #PWR0231
@@
 Wire Wire Line
 	18800 10550 18900 10550
-$Comp
-L power:+3V3 #PWR0230
-U 1 1 5DE91950
-P 18600 10250
-F 0 "#PWR0230" H 18600 10100 50  0001 C CNN
-F 1 "+3V3" V 18615 10378 50  0000 L CNN
-F 2 "" H 18600 10250 50  0001 C CNN
-F 3 "" H 18600 10250 50  0001 C CNN
-	1    18600 10250
-	0    -1   -1   0
-$EndComp
-Wire Wire Line
-	18600 10250 18900 10250
 Text GLabel 15050 2900 0    50   Output ~ 0
 DDR3_Vtt_EN
@@
 Wire Wire Line
 	20850 1200 20850 1350
+Wire Wire Line
+	21100 9650 21200 9650
+Wire Wire Line
+	21200 9650 21200 9550
+Text Label 22000 9650 2    50   ~ 0
+FLASH_~CS
+Wire Wire Line
+	18150 10350 18900 10350
+$Comp
+L power:+3V3 #PWR?
+U 1 1 60B148AD
+P 18900 10200
+F 0 "#PWR?" H 18900 10050 50  0001 C CNN
+F 1 "+3V3" H 18915 10373 50  0000 C CNN
+F 2 "" H 18900 10200 50  0001 C CNN
+F 3 "" H 18900 10200 50  0001 C CNN
+	1    18900 10200
+	1    0    0    -1
+$EndComp
+Wire Wire Line
+	18900 10200 18900 10250
+Text Label 18150 10450 0    50   ~ 0
+FLASH_CLK
+Wire Wire Line
+	18150 10450 18900 10450
+Wire Wire Line
+	21500 9550 21500 9850
+Wire Wire Line
+	21500 9850 21100 9850
+Wire Wire Line
+	21200 9650 22000 9650
+Connection ~ 21200 9650
+Wire Wire Line
+	21500 9850 22000 9850
+Connection ~ 21500 9850
+Wire Wire Line
+	19600 8900 19600 8800
+Wire Wire Line
+	20600 9350 20600 9250
+Wire Wire Line
+	20600 9250 21200 9250
+Connection ~ 22150 9250
+Wire Wire Line
+	22150 9250 22150 9600
+Wire Wire Line
+	21200 9350 21200 9250
+Connection ~ 21200 9250
+Wire Wire Line
+	21200 9250 21500 9250
+Wire Wire Line
+	21500 9350 21500 9250
+Connection ~ 21500 9250
+Wire Wire Line
+	21500 9250 22150 9250
+Wire Wire Line
+	20600 10150 22150 10150
+Wire Wire Line
+	22150 9800 22150 10150
+Connection ~ 22150 10150
+Wire Wire Line
+	20100 9650 19600 9650
+Connection ~ 19600 9650
+Wire Wire Line
+	20100 9550 19500 9550
+Connection ~ 19500 9550
+Text Label 18150 9650 0    50   ~ 0
+FLASH_D1
+Text Label 18150 9550 0    50   ~ 0
+FLASH_D0
+Wire Wire Line
+	19600 9650 18150 9650
+Wire Wire Line
+	19500 9550 18150 9550
+Wire Wire Line
+	19500 9550 19500 10250
+Wire Wire Line
+	19600 9650 19600 10350
+Wire Wire Line
+	19700 9850 20100 9850
+Wire Wire Line
+	19800 9950 20100 9950
+$Comp
+L Memory_Flash:W25Q128JVS U27
+U 1 1 5FF23C0A
+P 20600 9750
+F 0 "U27" H 20950 10100 50  0000 C CNN
+F 1 "W25Q128JVS" H 20300 10100 50  0000 C CNN
+F 2 "Package_SO:SOIC-8_5.23x5.23mm_P1.27mm" H 20600 9750 50  0001 C CNN
+F 3 "http://www.winbond.com/resource-files/w25q128jv_dtr%20revc%2003272018%20plus.pdf" H 20600 9750 50  0001 C CNN
+	1    20600 9750
+	-1   0    0    -1
+$EndComp
 $EndSCHEMATC
