File: hardware/ecp5_mainboard/power.sch (KiCad schematic (older format))
At the start: 112 parts, among them J1 12V_EXT, J15 PWR, Q1 BSH111BKR, Q2 BC850, Q3 BSH111BKR, Q4 BC850, Q5 BSH111BKR, Q6 BSH111BKR, Q7 BSH111BKR, Q8 BSH111BKR, U1 MAX811MEUS-T, U10 TPS62823, U2 LM3880, U3 TLV75712PDR, U4 TPS565208, U5 LM21212-2, U6 TLV75712PDR, U7 TPS62823, U8 TPS62823, U9 TPS62823

Commit message: U4 changed to upstream symbol
Parts:
- removed U4: TPS565208, Package_TO_SOT_SMD:SOT-23-6, symbol eco_power:TPS565208
- added U4: TPS565208, Package_TO_SOT_SMD:SOT-23-6, symbol Regulator_Switching:TPS565208
Changed lines of the file:
@@
 EESchema Schematic File Version 4
 LIBS:ecp5_mainboard-cache
-EELAYER 29 0
+EELAYER 30 0
 EELAYER END
 $Descr A3 16535 11693
@@
 Wire Wire Line
 	4550 2650 4550 2750
-$Comp
-L eco_power:TPS565208 U4
-U 1 1 5B5E5433
-P 6150 2750
-F 0 "U4" H 6150 3215 50  0000 C CNN
-F 1 "TPS565208" H 6150 3124 50  0000 C CNN
-F 2 "Package_TO_SOT_SMD:SOT-23-6" H 6150 2750 50  0001 C CNN
-F 3 "http://www.ti.com/lit/ds/symlink/tps565208.pdf" H 6150 2750 50  0001 C CNN
-	1    6150 2750
-	1    0    0    -1
-$EndComp
-Wire Wire Line
-	5450 2750 5350 2750
-Wire Wire Line
-	5350 2750 5350 2550
 Connection ~ 4550 2400
-Wire Wire Line
-	5450 2550 5350 2550
-Wire Wire Line
-	5450 2950 5350 2950
-Wire Wire Line
-	5350 2950 5350 3350
-Wire Wire Line
-	5350 3350 5050 3350
 Connection ~ 4550 3350
 $Comp
@@
 Wire Wire Line
 	5050 3350 4550 3350
-Wire Wire Line
-	7150 2200 7150 2550
-Wire Wire Line
-	7150 2550 6850 2550
 $Comp
 L Device:C_Small C8
@@
 $EndComp
 Wire Wire Line
-	7150 2550 7150 2750
-Wire Wire Line
 	7150 2750 7100 2750
-Connection ~ 7150 2550
-Wire Wire Line
-	6900 2750 6850 2750
 $Comp
 L Device:R_Small R12
@@
 	8300 2350 8300 2200
 Wire Wire Line
-	8300 2550 8300 2950
-Wire Wire Line
-	8300 2950 6850 2950
+	8300 2550 8300 2850
 $Comp
 L Device:R_Small R13
@@
 	1    0    0    -1
 $EndComp
-Wire Wire Line
-	8300 3050 8300 2950
-Connection ~ 8300 2950
-Wire Wire Line
-	5350 3350 8300 3350
 Wire Wire Line
 	8300 3350 8300 3250
@@
 	0    -1   -1   0
 $EndComp
-Wire Wire Line
-	5350 2550 5350 2400
-Wire Wire Line
-	5350 2400 5050 2400
-Connection ~ 5350 2550
 Connection ~ 5050 2400
 Wire Wire Line
@@
 $EndComp
 Connection ~ 8300 3350
-Connection ~ 5350 3350
 Text Label 2150 6400 0    50   ~ 0
 PWR_EN
@@
 U 1 1 5C219D75
 P 3200 2750
+AR Path="/5C219D75" Ref="D3"  Part="1"
+AR Path="/5B5D9B41/5C219D75" Ref="D3"  Part="1"
 F 0 "D3" V 3179 2890 50  0000 L CNN
 F 1 "MBR15U60" V 3270 2890 50  0000 L CNN
@@
 	9000 2550 9000 2400
 Connection ~ 9000 2400
+$Comp
+L Regulator_Switching:TPS565208 U4
+U 1 1 5DB6D21A
+P 6150 2750
+F 0 "U4" H 6150 3117 50  0000 C CNN
+F 1 "TPS565208" H 6150 3026 50  0000 C CNN
+F 2 "Package_TO_SOT_SMD:SOT-23-6" H 6200 2500 50  0001 L CNN
+F 3 "http://www.ti.com/lit/ds/symlink/tps565208.pdf" H 6150 2750 50  0001 C CNN
+	1    6150 2750
+	1    0    0    -1
+$EndComp
+Wire Wire Line
+	5050 3350 6150 3350
+Wire Wire Line
+	5600 2400 5600 2650
+Wire Wire Line
+	5600 2650 5750 2650
+Wire Wire Line
+	5050 2400 5600 2400
+Wire Wire Line
+	5600 2650 5600 2850
+Wire Wire Line
+	5600 2850 5750 2850
+Connection ~ 5600 2650
+Wire Wire Line
+	6150 3050 6150 3350
+Connection ~ 6150 3350
+Wire Wire Line
+	6150 3350 8300 3350
+Wire Wire Line
+	6550 2850 8300 2850
+Connection ~ 8300 2850
+Wire Wire Line
+	8300 2850 8300 3050
+Wire Wire Line
+	7150 2200 7150 2750
+Wire Wire Line
+	6550 2750 6900 2750
+Wire Wire Line
+	6550 2650 6700 2650
+Wire Wire Line
+	6700 2650 6700 2200
+Wire Wire Line
+	6700 2200 7150 2200
+Connection ~ 7150 2200
 $EndSCHEMATC

Commit message: U3, U6 changed to upstream KiCAD symbols
Parts:
- removed U3, U6: TLV75712PDR, Custom Parts:TI_WSON8_2x2mm_p0.65mm, symbol eco_power:TLV75712PDR
- added U3, U6: TLV75712PDRV, Package_SON:WSON-6-1EP_2x2mm_P0.65mm_EP1x1.6mm, symbol Regulator_Linear:TLV75712PDRV
Connections:
- wire segments 446 -> 440
Changed lines of the file:
@@
 	8250 7000 7950 7000
-$Comp
-L eco_power:TLV75712PDR U3
-U 1 1 5C1EB81E
-P 4100 9850
-F 0 "U3" H 4100 10315 50  0000 C CNN
-F 1 "TLV75712PDR" H 4100 10224 50  0000 C CNN
-F 2 "Custom Parts:TI_WSON8_2x2mm_p0.65mm" H 4100 9850 50  0001 C CNN
-F 3 "" H 4100 9850 50  0001 C CNN
-	1    4100 9850
-	1    0    0    -1
-$EndComp
 $Comp
 L power:+2V5 #PWR06
@@
 Wire Wire Line
 	2800 9450 2800 9650
-Wire Wire Line
-	2800 9850 3400 9850
-Wire Wire Line
-	3400 9650 2800 9650
 Connection ~ 2800 9650
 Wire Wire Line
-	2800 9650 2800 9850
+	2800 9650 2800 9750
 $Comp
 L Device:C_Small C1
@@
 $EndComp
 Wire Wire Line
-	2800 9850 2800 9950
-Connection ~ 2800 9850
-Wire Wire Line
 	2800 10150 2800 10450
-Wire Wire Line
-	2800 10450 3300 10450
-Wire Wire Line
-	4100 10450 4100 10350
-Wire Wire Line
-	3400 10050 3300 10050
-Wire Wire Line
-	3300 10050 3300 10450
-Connection ~ 3300 10450
-Wire Wire Line
-	3300 10450 4100 10450
 $Comp
 L power:GND #PWR012
@@
 Wire Wire Line
 	5000 9450 5000 9650
-Wire Wire Line
-	5000 9650 4800 9650
 $Comp
 L Device:C_Small C5
@@
 1.2V/1A\nSERDES analog
 $Comp
-L eco_power:TLV75712PDR U6
-U 1 1 5C5AEF13
-P 8850 9900
-F 0 "U6" H 8850 10365 50  0000 C CNN
-F 1 "TLV75712PDR" H 8850 10274 50  0000 C CNN
-F 2 "Custom Parts:TI_WSON8_2x2mm_p0.65mm" H 8850 9900 50  0001 C CNN
-F 3 "" H 8850 9900 50  0001 C CNN
-	1    8850 9900
-	1    0    0    -1
-$EndComp
-$Comp
 L power:+2V5 #PWR020
 U 1 1 5C5AEF1A
@@
 Wire Wire Line
 	7550 9500 7550 9700
-Wire Wire Line
-	7550 9900 8150 9900
-Wire Wire Line
-	8150 9700 7550 9700
 Connection ~ 7550 9700
 Wire Wire Line
-	7550 9700 7550 9900
+	7550 9700 7550 9800
 $Comp
 L Device:C_Small C10
@@
 $EndComp
 Wire Wire Line
-	7550 9900 7550 10000
-Connection ~ 7550 9900
-Wire Wire Line
 	7550 10200 7550 10500
-Wire Wire Line
-	7550 10500 8050 10500
-Wire Wire Line
-	8850 10500 8850 10400
-Wire Wire Line
-	8150 10100 8050 10100
-Wire Wire Line
-	8050 10100 8050 10500
-Connection ~ 8050 10500
-Wire Wire Line
-	8050 10500 8850 10500
 $Comp
 L power:GND #PWR024
@@
 Wire Wire Line
 	9750 9500 9750 9700
-Wire Wire Line
-	9750 9700 9550 9700
 $Comp
 L Device:C_Small C14
@@
 	6700 2200 7150 2200
 Connection ~ 7150 2200
+$Comp
+L Regulator_Linear:TLV75712PDRV U3
+U 1 1 5DA22C23
+P 4100 9750
+F 0 "U3" H 3950 10000 50  0000 C CNN
+F 1 "TLV75712PDRV" H 4400 10000 50  0000 C CNN
+F 2 "Package_SON:WSON-6-1EP_2x2mm_P0.65mm_EP1x1.6mm" H 4100 10075 50  0001 C CIN
+F 3 "https://www.ti.com/lit/ds/symlink/tlv757p.pdf" H 4100 9800 50  0001 C CNN
+	1    4100 9750
+	1    0    0    -1
+$EndComp
+$Comp
+L Regulator_Linear:TLV75712PDRV U6
+U 1 1 5DA248CB
+P 8850 9800
+F 0 "U6" H 8700 10050 50  0000 C CNN
+F 1 "TLV75712PDRV" H 9150 10050 50  0000 C CNN
+F 2 "Package_SON:WSON-6-1EP_2x2mm_P0.65mm_EP1x1.6mm" H 8850 10125 50  0001 C CIN
+F 3 "https://www.ti.com/lit/ds/symlink/tlv757p.pdf" H 8850 9850 50  0001 C CNN
+	1    8850 9800
+	1    0    0    -1
+$EndComp
+Wire Wire Line
+	2800 10450 4100 10450
+Wire Wire Line
+	4100 10050 4100 10450
+Wire Wire Line
+	2800 9650 3800 9650
+Wire Wire Line
+	3800 9750 2800 9750
+Connection ~ 2800 9750
+Wire Wire Line
+	2800 9750 2800 9950
+Wire Wire Line
+	4400 9650 5000 9650
+Wire Wire Line
+	7550 10500 8850 10500
+Wire Wire Line
+	9150 9700 9750 9700
+Wire Wire Line
+	8850 10100 8850 10500
+Wire Wire Line
+	8550 9800 7550 9800
+Connection ~ 7550 9800
+Wire Wire Line
+	7550 9700 8550 9700
+Wire Wire Line
+	7550 9800 7550 10000
 $EndSCHEMATC

Commit message: J1 changed to KiCAD upstream symbol
Parts:
- removed J1: 12V_EXT, Connector_BarrelJack:BarrelJack_Horizontal, symbol ecp5_mainboard-rescue:Barrel_Jack-Connector
- added J1: 12V_EXT, symbol Connector:Barrel_Jack_Switch
Changed lines of the file:
@@
 Comment4 ""
 $EndDescr
-$Comp
-L ecp5_mainboard-rescue:Barrel_Jack-Connector J1
-U 1 1 5B5D9C9C
-P 1950 2650
-F 0 "J1" H 2028 2975 50  0000 C CNN
-F 1 "12V_EXT" H 2028 2884 50  0000 C CNN
-F 2 "Connector_BarrelJack:BarrelJack_Horizontal" H 2000 2610 50  0001 C CNN
-F 3 "~" H 2000 2610 50  0001 C CNN
-	1    1950 2650
-	1    0    0    -1
-$EndComp
 Text GLabel 1600 3600 0    50   Input ~ 0
 PCIe_12V
@@
 Wire Wire Line
 	7550 9800 7550 10000
+$Comp
+L Connector:Barrel_Jack_Switch J1
+U 1 1 5DA5AC57
+P 1950 2650
+F 0 "J1" H 2007 2967 50  0000 C CNN
+F 1 "12V_EXT" H 2007 2876 50  0000 C CNN
+F 2 "" H 2000 2610 50  0001 C CNN
+F 3 "~" H 2000 2610 50  0001 C CNN
+	1    1950 2650
+	1    0    0    -1
+$EndComp
 $EndSCHEMATC
