File: hardware/ecp5_mainboard/power.sch (KiCad schematic (older format))
At the start: 112 parts, among them J1 12V_EXT, J15 PWR, Q1 BSH111BKR, Q2 BC850, Q3 BSH111BKR, Q4 BC850, Q5 BSH111BKR, Q6 BSH111BKR, Q7 BSH111BKR, Q8 BSH111BKR, U1 MAX811MEUS-T, U10 TPS62823, U2 LM3880, U3 TLV75712PDRV, U4 TPS565208, U5 LM21212-2, U6 TLV75712PDRV, U7 TPS62823, U8 TPS62823, U9 TPS62823

Commit message: U7-U10 changed to upstream TPS62823DLC
Parts:
- removed U10, U7, U8, U9: TPS62823, Custom Parts:TI_VSON-HR_1.5x2mm_p0.5mm, symbol eco_power:TPS62823
- added U10, U7, U8, U9: TPS62823DLC, Package_DFN_QFN:Texas_VSON-HR-8_1.5x2mm_P0.5mm, symbol Regulator_Switching:TPS62823DLC
Connections:
- wire segments 440 -> 428
Other:
- moved on the sheet: C15, C16, C17, C18, R26, R27, R28, R29, TP10, TP11, TP12, TP9
