File: hardware/ecp5_mainboard/debug.sch (KiCad schematic (older format))
At the start: 34 parts, among them J2 USB_C_Receptacle, U12 93AA46B_OT, U13 FT2232H, X1 12MHz

Commit message: U12 changed to upstream symbol
Parts:
- removed U12: 93AA46B_OT, Package_TO_SOT_SMD:SOT-23-6, symbol eco_memory:93AA46B_OT
- added U12: 93AAxxBT-xOT, Package_TO_SOT_SMD:SOT-23-6, symbol Memory_EEPROM:93AAxxBT-xOT
Connections:
- net labels added: CS
Changed lines of the file:
@@
 EESchema Schematic File Version 4
 LIBS:ecp5_mainboard-cache
-EELAYER 29 0
+EELAYER 30 0
 EELAYER END
 $Descr A4 11693 8268
@@
 Connection ~ 7600 6300
 $Comp
-L eco_memory:93AA46B_OT U12
-U 1 1 628C86C1
-P 5150 5400
-F 0 "U12" H 5150 5815 50  0000 C CNN
-F 1 "93AA46B_OT" H 5150 5724 50  0000 C CNN
-F 2 "Package_TO_SOT_SMD:SOT-23-6" H 5150 5400 50  0001 C CNN
-F 3 "http://ww1.microchip.com/downloads/en/DeviceDoc/20001749K.pdf" H 5150 5400 50  0001 C CNN
-	1    5150 5400
-	-1   0    0    -1
-$EndComp
-$Comp
 L power:+3V3 #PWR069
 U 1 1 628D3E7E
@@
 $EndComp
 Wire Wire Line
-	4050 5750 4050 5550
-Wire Wire Line
-	4050 5550 4450 5550
-Wire Wire Line
 	4050 5000 4050 5100
-Wire Wire Line
-	4050 5250 4450 5250
 $Comp
 L Device:C_Small C87
@@
 $EndComp
 Wire Wire Line
-	4050 5300 4050 5250
-Connection ~ 4050 5250
-Wire Wire Line
-	4050 5550 4050 5500
-Connection ~ 4050 5550
-Wire Wire Line
-	5850 5250 5900 5250
-Wire Wire Line
-	5900 5250 5900 4650
-Wire Wire Line
-	5900 4650 7000 4650
-Wire Wire Line
-	5850 5350 6000 5350
-Wire Wire Line
 	6000 5350 6000 4750
 Wire Wire Line
@@
 Wire Wire Line
 	6400 4850 6400 5450
-Wire Wire Line
-	6400 5450 5850 5450
 $Comp
 L Device:R_Small R38
@@
 Connection ~ 4050 5100
 Wire Wire Line
-	4050 5100 4050 5250
-Wire Wire Line
 	5000 4750 4450 4750
 Wire Wire Line
@@
 	5400 4550 6100 4550
 Connection ~ 6100 5550
-Wire Wire Line
-	6100 5550 5850 5550
-Wire Wire Line
-	5400 4650 5900 4650
-Connection ~ 5900 4650
 Wire Wire Line
 	6000 4750 5400 4750
@@
 NoConn ~ 3200 3450
 NoConn ~ 3200 3550
+$Comp
+L Memory_EEPROM:93AAxxBT-xOT U12
+U 1 1 5DF25CEE
+P 5250 5450
+F 0 "U12" H 5000 5700 50  0000 C CNN
+F 1 "93AAxxBT-xOT" H 5550 5700 50  0000 C CNN
+F 2 "Package_TO_SOT_SMD:SOT-23-6" H 5300 5800 50  0001 C CNN
+F 3 "http://ww1.microchip.com/downloads/en/DeviceDoc/20001749K.pdf" H 5250 5450 50  0001 C CNN
+	1    5250 5450
+	1    0    0    -1
+$EndComp
+Wire Wire Line
+	4050 5500 4050 5750
+Wire Wire Line
+	4050 5750 5250 5750
+Connection ~ 4050 5750
+Wire Wire Line
+	4450 5100 5250 5100
+Wire Wire Line
+	5250 5100 5250 5150
+Connection ~ 4450 5100
+Wire Wire Line
+	4050 5100 4050 5300
+Wire Wire Line
+	5650 5550 6100 5550
+Wire Wire Line
+	5650 5450 6400 5450
+Wire Wire Line
+	5650 5350 6000 5350
+Wire Wire Line
+	5400 4650 5900 4650
+Wire Wire Line
+	5900 4650 5900 5100
+Wire Wire Line
+	5900 5100 5750 5100
+Connection ~ 5900 4650
+Wire Wire Line
+	5900 4650 7000 4650
+Text Label 5750 5100 0    50   ~ 0
+CS
+Wire Wire Line
+	4850 5350 4700 5350
+Text Label 4700 5350 0    50   ~ 0
+CS
 $EndSCHEMATC

Commit message: U13 changed
Parts:
- removed U13: FT2232H, Package_QFP:LQFP-64_10x10mm_P0.5mm, symbol Interface_USB:FT2232H
- added U13: FT2232HL, Package_QFP:LQFP-64_10x10mm_P0.5mm, symbol Interface_USB:FT2232HL
Changed lines of the file:
@@
 EESchema Schematic File Version 4
-LIBS:ecp5_mainboard-cache
 EELAYER 30 0
 EELAYER END
@@
 Comment4 ""
 $EndDescr
-$Comp
-L Interface_USB:FT2232H U13
-U 1 1 627DD271
-P 8200 3950
-F 0 "U13" H 8200 4000 50  0000 C CNN
-F 1 "FT2232H" H 8200 3900 50  0000 C CNN
-F 2 "Package_QFP:LQFP-64_10x10mm_P0.5mm" H 8200 3950 50  0001 C CNN
-F 3 "http://www.ftdichip.com/Products/ICs/FT2232H.html" H 8200 3950 50  0001 C CNN
-	1    8200 3950
-	1    0    0    -1
-$EndComp
 Text Label 6550 5150 0    50   ~ 0
 FTDI_12MHz
@@
 Text Label 4700 5350 0    50   ~ 0
 CS
+$Comp
+L Interface_USB:FT2232HL U13
+U 1 1 5E9C83B5
+P 8200 3950
+F 0 "U13" H 8200 4000 50  0000 C CNN
+F 1 "FT2232HL" H 8200 3900 50  0000 C CNN
+F 2 "Package_QFP:LQFP-64_10x10mm_P0.5mm" H 8200 3950 50  0001 C CNN
+F 3 "https://www.ftdichip.com/Support/Documents/DataSheets/ICs/DS_FT2232H.pdf" H 8200 3950 50  0001 C CNN
+	1    8200 3950
+	1    0    0    -1
+$EndComp
 $EndSCHEMATC
