File: hardware/ecp5_mainboard/ports.sch (KiCad schematic (older format))
At the start: 98 parts, among them J13 Micro_SD_Card, J3 HDMI_A, J4 USB_A, P4 JK0654219NL, U17 TPS2041B, U18 PCA9306, U19 TFP410, U20 TPS2041B, U21 KSZ9031RNXCA, U22 USB3300-EZK, Y2 25MHz, Y3 24MHz

Commit message: U21 symbol changed to symbol from KiCAD library
Parts:
- U21: symbol ecp5_mainboard-rescue:KSZ9031RNXCA-Interface_Ethernet -> Interface_Ethernet:KSZ9031RNXCA
Changed lines of the file:
@@
 EESchema Schematic File Version 4
 LIBS:ecp5_mainboard-cache
-EELAYER 29 0
+EELAYER 26 0
 EELAYER END
 $Descr A3 16535 11693
@@
 $EndDescr
 $Comp
-L ecp5_mainboard-rescue:KSZ9031RNXCA-Interface_Ethernet U21
+L Interface_Ethernet:KSZ9031RNXCA U21
 U 1 1 5CA0A635
 P 11450 3250
-F 0 "U21" H 11250 1700 50  0000 C CNN
-F 1 "KSZ9031RNXCA" H 11000 1800 50  0000 C CNN
+F 0 "U21" H 12595 4875 50  0000 C CNN
+F 1 "KSZ9031RNXCA" H 12810 4800 50  0000 C CNN
 F 2 "Package_DFN_QFN:QFN-48-1EP_7x7mm_P0.5mm_EP5.15x5.15mm" H 11900 1800 50  0001 L CNN
 F 3 "http://ww1.microchip.com/downloads/en/DeviceDoc/00002117C.pdf" H 11450 1500 50  0001 C CNN
@@
 U 1 1 5CDDA130
 P 15100 3300
-F 0 "RN5" V 14683 3300 50  0000 C CNN
-F 1 "10k" V 14774 3300 50  0000 C CNN
+F 0 "RN5" V 15400 3295 50  0000 C CNN
+F 1 "10k" V 15310 3300 50  0000 C CNN
 F 2 "Resistor_SMD:R_Array_Convex_4x0402" V 15375 3300 50  0001 C CNN
 F 3 "~" H 15100 3300 50  0001 C CNN

Commit message: J13 changed to KiCAD upstream symbol
Parts:
- removed J13: Micro_SD_Card, Connector_Card:microSD_HC_Hirose_DM3AT-SF-PEJM5, symbol ecp5_mainboard-rescue:Micro_SD_Card-Connector
- added J13: Micro_SD_Card, symbol Connector:Micro_SD_Card
Changed lines of the file:
@@
 EESchema Schematic File Version 4
 LIBS:ecp5_mainboard-cache
-EELAYER 26 0
+EELAYER 30 0
 EELAYER END
 $Descr A3 16535 11693
@@
 	13650 750  14000 750
 $Comp
-L ecp5_mainboard-rescue:Micro_SD_Card-Connector J13
-U 1 1 632D42B7
-P 1550 1550
-AR Path="/632D42B7" Ref="J13"  Part="1"
-AR Path="/5CA09014/632D42B7" Ref="J13"  Part="1"
-F 0 "J13" H 1500 2267 50  0000 C CNN
-F 1 "Micro_SD_Card" H 1500 2176 50  0000 C CNN
-F 2 "Connector_Card:microSD_HC_Hirose_DM3AT-SF-PEJM5" H 2700 1850 50  0001 C CNN
-F 3 "http://katalog.we-online.de/em/datasheet/693072010801.pdf" H 1550 1550 50  0001 C CNN
-	1    1550 1550
-	-1   0    0    -1
-$EndComp
-$Comp
 L power:GND #PWR0249
 U 1 1 632D4719
@@
 Text Label 9800 3750 0    50   ~ 0
 MX2+
+$Comp
+L Connector:Micro_SD_Card J13
+U 1 1 5DB53AEA
+P 1550 1550
+F 0 "J13" H 1500 2267 50  0000 C CNN
+F 1 "Micro_SD_Card" H 1500 2176 50  0000 C CNN
+F 2 "" H 2700 1850 50  0001 C CNN
+F 3 "http://katalog.we-online.de/em/datasheet/693072010801.pdf" H 1550 1550 50  0001 C CNN
+	1    1550 1550
+	-1   0    0    -1
+$EndComp
 $EndSCHEMATC

Commit message: P4 changed to upstream KiCAD symbol
Parts:
- removed P4: JK0654219NL, Custom Parts:Pulse_MagJack_JK0654219NL, symbol eco_connectors:JK0654219
- added P4: JK0654219, Connector_RJ:RJ45_Pulse_JK0654219NL_Horizontal, symbol Connector:JK0654219
Connections:
- wire segments 661 -> 658
Other:
- moved on the sheet: R63, R64
Changed lines of the file:
@@
 	11450 5000 11450 4850
 Connection ~ 11400 5000
-$Comp
-L eco_connectors:JK0654219 P4
-U 1 1 5CA2589B
-P 5300 1700
-F 0 "P4" H 5194 2765 50  0000 C CNN
-F 1 "JK0654219NL" H 5194 2674 50  0000 C CNN
-F 2 "Custom Parts:Pulse_MagJack_JK0654219NL" H 6450 1400 50  0001 C CNN
-F 3 "" H 6450 1400 50  0001 C CNN
-	1    5300 1700
-	-1   0    0    -1
-$EndComp
-Wire Wire Line
-	6100 1400 7250 1400
-Wire Wire Line
-	6100 1600 7250 1600
 Text Label 7250 1400 2    50   ~ 0
 MX1+
 Text Label 7250 1600 2    50   ~ 0
 MX1-
-Wire Wire Line
-	6100 1800 7250 1800
-Wire Wire Line
-	6100 2000 7250 2000
 Text Label 7250 1800 2    50   ~ 0
 MX2+
@@
 	1    0    0    -1
 $EndComp
-Wire Wire Line
-	6100 2200 7250 2200
-Wire Wire Line
-	6100 2400 7250 2400
 Text Label 7250 2200 2    50   ~ 0
 MX3+
 Text Label 7250 2400 2    50   ~ 0
 MX3-
-Wire Wire Line
-	6100 2600 7250 2600
-Wire Wire Line
-	6100 2800 7250 2800
 Text Label 7250 2600 2    50   ~ 0
 MX4+
@@
 	6200 3000 6200 1500
 Wire Wire Line
-	6200 1500 6100 1500
-Wire Wire Line
-	6100 1900 6350 1900
-Wire Wire Line
 	6350 1900 6350 3000
 Wire Wire Line
 	6500 3000 6500 2300
 Wire Wire Line
-	6500 2300 6100 2300
-Wire Wire Line
-	6100 2700 6650 2700
-Wire Wire Line
 	6650 2700 6650 3000
 Wire Wire Line
@@
 	6200 3400 6200 3300
 Connection ~ 6200 3300
-Wire Wire Line
-	6200 3300 5300 3300
-Wire Wire Line
-	5300 3300 5300 3200
 Text Label 9800 3150 0    50   ~ 0
 MX4+
@@
 Wire Wire Line
 	15650 3850 15300 3850
-Text Label 7100 900  2    50   ~ 0
-ETH_LED1
-$Comp
-L Device:R_Small R63
-U 1 1 5CF7CC99
-P 6300 900
-F 0 "R63" V 6200 900 50  0000 C CNN
-F 1 "1k" V 6300 900 50  0000 C CNN
-F 2 "Resistor_SMD:R_0402_1005Metric" H 6300 900 50  0001 C CNN
-F 3 "~" H 6300 900 50  0001 C CNN
-	1    6300 900
-	0    1    1    0
-$EndComp
-$Comp
-L Device:R_Small R64
-U 1 1 5CF8D044
-P 6300 1100
-F 0 "R64" V 6200 1100 50  0000 C CNN
-F 1 "1k" V 6300 1100 50  0000 C CNN
-F 2 "Resistor_SMD:R_0402_1005Metric" H 6300 1100 50  0001 C CNN
-F 3 "~" H 6300 1100 50  0001 C CNN
-	1    6300 1100
-	0    1    1    0
-$EndComp
-Wire Wire Line
-	6200 900  6100 900
-Wire Wire Line
-	6100 1100 6200 1100
-Wire Wire Line
-	6400 900  7100 900
-Text Label 7100 1100 2    50   ~ 0
-ETH_LED2
-Wire Wire Line
-	7100 1100 6400 1100
-$Comp
-L power:GND #PWR0123
-U 1 1 5CFD0222
-P 6200 1300
-F 0 "#PWR0123" H 6200 1050 50  0001 C CNN
-F 1 "GND" V 6205 1172 50  0000 R CNN
-F 2 "" H 6200 1300 50  0001 C CNN
-F 3 "" H 6200 1300 50  0001 C CNN
-	1    6200 1300
-	0    -1   -1   0
-$EndComp
-Wire Wire Line
-	6200 1300 6150 1300
-Wire Wire Line
-	6150 1300 6150 1200
-Wire Wire Line
-	6150 1000 6100 1000
-Wire Wire Line
-	6100 1200 6150 1200
-Connection ~ 6150 1200
-Wire Wire Line
-	6150 1200 6150 1000
 $Comp
 L Connector:USB_A J4
@@
 	-1   0    0    -1
 $EndComp
+$Comp
+L Connector:JK0654219 P4
+U 1 1 5DC3A4F4
+P 4800 2100
+F 0 "P4" H 5345 3250 50  0000 C CNN
+F 1 "JK0654219" H 4410 3255 50  0000 C CNN
+F 2 "Connector_RJ:RJ45_Pulse_JK0654219NL_Horizontal" H 4795 805 50  0001 C CNN
+F 3 "https://media.digikey.com/pdf/Data%20Sheets/Pulse%20PDFs/JK%20Series.pdf" H 4795 805 50  0001 C CNN
+	1    4800 2100
+	-1   0    0    -1
+$EndComp
+Wire Wire Line
+	5500 3000 5600 3000
+$Comp
+L Device:R_Small R64
+U 1 1 5CF8D044
+P 5700 3000
+F 0 "R64" V 5600 3000 50  0000 C CNN
+F 1 "1k" V 5700 3000 50  0000 C CNN
+F 2 "Resistor_SMD:R_0402_1005Metric" H 5700 3000 50  0001 C CNN
+F 3 "~" H 5700 3000 50  0001 C CNN
+	1    5700 3000
+	0    1    1    0
+$EndComp
+Text Label 6150 3000 2    50   ~ 0
+ETH_LED2
+Wire Wire Line
+	6150 3000 5800 3000
+Wire Wire Line
+	6200 3300 5500 3300
+Wire Wire Line
+	5500 3100 5500 3300
+Connection ~ 5500 3300
+Wire Wire Line
+	5500 3300 4800 3300
+Wire Wire Line
+	5600 1100 5500 1100
+$Comp
+L Device:R_Small R63
+U 1 1 5CF7CC99
+P 5700 1100
+F 0 "R63" V 5600 1100 50  0000 C CNN
+F 1 "1k" V 5700 1100 50  0000 C CNN
+F 2 "Resistor_SMD:R_0402_1005Metric" H 5700 1100 50  0001 C CNN
+F 3 "~" H 5700 1100 50  0001 C CNN
+	1    5700 1100
+	0    1    1    0
+$EndComp
+Text Label 6150 1100 2    50   ~ 0
+ETH_LED1
+$Comp
+L power:GND #PWR0123
+U 1 1 5CFD0222
+P 5750 1200
+F 0 "#PWR0123" H 5750 950 50  0001 C CNN
+F 1 "GND" H 5850 1050 50  0000 R CNN
+F 2 "" H 5750 1200 50  0001 C CNN
+F 3 "" H 5750 1200 50  0001 C CNN
+	1    5750 1200
+	1    0    0    -1
+$EndComp
+Wire Wire Line
+	5500 1200 5750 1200
+Wire Wire Line
+	5800 1100 6150 1100
+Wire Wire Line
+	5500 1400 7250 1400
+Wire Wire Line
+	5500 1500 6200 1500
+Wire Wire Line
+	5500 1600 7250 1600
+Wire Wire Line
+	5500 1800 7250 1800
+Wire Wire Line
+	5500 1900 6350 1900
+Wire Wire Line
+	5500 2000 7250 2000
+Wire Wire Line
+	5500 2200 7250 2200
+Wire Wire Line
+	5500 2300 6500 2300
+Wire Wire Line
+	5500 2400 7250 2400
+Wire Wire Line
+	5500 2600 7250 2600
+Wire Wire Line
+	5500 2700 6650 2700
+Wire Wire Line
+	5500 2800 7250 2800
 $EndSCHEMATC

Commit message: DA1-DA6 changed to upstream symbol TPD4E02B04DQA
Parts:
- removed DA5, DA6: TPD4E02B04, Custom Parts:USON10, symbol eco_interface:TPD4E02B04
- added DA5, DA6: TPD4E02B04DQA, Package_SON:USON-10_2.5x1.0mm_P0.5mm, symbol Power_Protection:TPD4E02B04DQA
Connections:
- wire segments 658 -> 630
Changed lines of the file:
@@
 EESchema Schematic File Version 4
-LIBS:ecp5_mainboard-cache
 EELAYER 30 0
 EELAYER END
@@
 Text Label 1950 5900 1    50   ~ 0
 HDMI_5V
-$Comp
-L eco_interface:TPD4E02B04 DA5
-U 1 1 6003247F
-P 4800 4450
-F 0 "DA5" H 4800 5237 60  0000 C CNN
-F 1 "TPD4E02B04" H 4800 5131 60  0000 C CNN
-F 2 "Custom Parts:USON10" H 4800 4450 60  0001 C CNN
-F 3 "" H 4800 4450 60  0001 C CNN
-	1    4800 4450
-	1    0    0    -1
-$EndComp
-Text Label 3800 4000 0    50   ~ 0
+Text Label 4000 4200 0    50   ~ 0
 TMDS_D2+
-Wire Wire Line
-	3800 4000 4250 4000
-Wire Wire Line
-	4350 4100 4250 4100
-Wire Wire Line
-	4250 4100 4250 4000
-Connection ~ 4250 4000
-Wire Wire Line
-	4250 4000 4350 4000
-Text Label 3800 4300 0    50   ~ 0
+Text Label 4000 4300 0    50   ~ 0
 TMDS_D2-
-Wire Wire Line
-	3800 4300 4250 4300
-Wire Wire Line
-	4350 4400 4250 4400
-Wire Wire Line
-	4250 4400 4250 4300
-Connection ~ 4250 4300
-Wire Wire Line
-	4250 4300 4350 4300
-Text Label 3800 4600 0    50   ~ 0
+Text Label 4000 4500 0    50   ~ 0
 TMDS_D1+
-Wire Wire Line
-	3800 4600 4250 4600
-Wire Wire Line
-	4350 4700 4250 4700
-Wire Wire Line
-	4250 4700 4250 4600
-Connection ~ 4250 4600
-Wire Wire Line
-	4250 4600 4350 4600
-Text Label 3800 4900 0    50   ~ 0
+Text Label 4000 4600 0    50   ~ 0
 TMDS_D1-
 Wire Wire Line
-	3800 4900 4250 4900
-Wire Wire Line
-	4350 5000 4250 5000
-Wire Wire Line
-	4250 5000 4250 4900
-Connection ~ 4250 4900
-Wire Wire Line
-	4250 4900 4350 4900
-$Comp
-L power:GND #PWR0121
-U 1 1 6028ED65
-P 5400 5100
-F 0 "#PWR0121" H 5400 4850 50  0001 C CNN
-F 1 "GND" H 5405 4927 50  0000 C CNN
-F 2 "" H 5400 5100 50  0001 C CNN
-F 3 "" H 5400 5100 50  0001 C CNN
-	1    5400 5100
-	1    0    0    -1
-$EndComp
-Wire Wire Line
-	5400 5100 5400 5000
-Wire Wire Line
-	5400 4900 5250 4900
-Wire Wire Line
-	5250 5000 5400 5000
-Connection ~ 5400 5000
-Wire Wire Line
-	5400 5000 5400 4900
-$Comp
-L eco_interface:TPD4E02B04 DA6
-U 1 1 60363A81
-P 6500 4450
-F 0 "DA6" H 6500 5237 60  0000 C CNN
-F 1 "TPD4E02B04" H 6500 5131 60  0000 C CNN
-F 2 "Custom Parts:USON10" H 6500 4450 60  0001 C CNN
-F 3 "" H 6500 4450 60  0001 C CNN
-	1    6500 4450
-	1    0    0    -1
-$EndComp
-Text Label 5500 4000 0    50   ~ 0
+	5200 4400 5050 4400
+Text Label 5700 4200 0    50   ~ 0
 TMDS_D0+
-Wire Wire Line
-	5500 4000 5950 4000
-Wire Wire Line
-	6050 4100 5950 4100
-Wire Wire Line
-	5950 4100 5950 4000
-Connection ~ 5950 4000
-Wire Wire Line
-	5950 4000 6050 4000
-Text Label 5500 4300 0    50   ~ 0
+Text Label 5700 4300 0    50   ~ 0
 TMDS_D0-
-Wire Wire Line
-	5500 4300 5950 4300
-Wire Wire Line
-	6050 4400 5950 4400
-Wire Wire Line
-	5950 4400 5950 4300
-Connection ~ 5950 4300
-Wire Wire Line
-	5950 4300 6050 4300
-Text Label 5500 4600 0    50   ~ 0
+Text Label 5700 4500 0    50   ~ 0
 TMDS_CLK+
-Wire Wire Line
-	5500 4600 5950 4600
-Wire Wire Line
-	6050 4700 5950 4700
-Wire Wire Line
-	5950 4700 5950 4600
-Connection ~ 5950 4600
-Wire Wire Line
-	5950 4600 6050 4600
-Text Label 5500 4900 0    50   ~ 0
+Text Label 5700 4600 0    50   ~ 0
 TMDS_CLK-
-Wire Wire Line
-	5500 4900 5950 4900
-Wire Wire Line
-	6050 5000 5950 5000
-Wire Wire Line
-	5950 5000 5950 4900
-Connection ~ 5950 4900
-Wire Wire Line
-	5950 4900 6050 4900
 $Comp
 L power:GND #PWR0125
 U 1 1 60363A9F
-P 7100 5100
-F 0 "#PWR0125" H 7100 4850 50  0001 C CNN
-F 1 "GND" H 7105 4927 50  0000 C CNN
-F 2 "" H 7100 5100 50  0001 C CNN
-F 3 "" H 7100 5100 50  0001 C CNN
-	1    7100 5100
+P 6900 4600
+F 0 "#PWR0125" H 6900 4350 50  0001 C CNN
+F 1 "GND" H 6905 4427 50  0000 C CNN
+F 2 "" H 6900 4600 50  0001 C CNN
+F 3 "" H 6900 4600 50  0001 C CNN
+	1    6900 4600
 	1    0    0    -1
 $EndComp
 Wire Wire Line
-	7100 5100 7100 5000
-Wire Wire Line
-	7100 4900 6950 4900
-Wire Wire Line
-	6950 5000 7100 5000
-Connection ~ 7100 5000
-Wire Wire Line
-	7100 5000 7100 4900
+	6900 4400 6750 4400
 $Comp
 L Interface:PCA9306 U18
@@
 Wire Wire Line
 	5500 2800 7250 2800
+$Comp
+L Power_Protection:TPD4E02B04DQA DA5
+U 1 1 62F90330
+P 4850 4400
+F 0 "DA5" V 4433 4450 50  0000 C CNN
+F 1 "TPD4E02B04DQA" V 4524 4450 50  0000 C CNN
+F 2 "Package_SON:USON-10_2.5x1.0mm_P0.5mm" H 5150 4400 50  0001 L CNN
+F 3 "http://www.ti.com/lit/ds/symlink/tpd4e02b04.pdf" H 4975 4725 50  0001 C CNN
+	1    4850 4400
+	0    -1   1    0
+$EndComp
+Wire Wire Line
+	4000 4200 4550 4200
+Wire Wire Line
+	4000 4300 4550 4300
+Wire Wire Line
+	4000 4500 4550 4500
+Wire Wire Line
+	4000 4600 4550 4600
+$Comp
+L power:GND #PWR0121
+U 1 1 6028ED65
+P 5200 4600
+F 0 "#PWR0121" H 5200 4350 50  0001 C CNN
+F 1 "GND" H 5205 4427 50  0000 C CNN
+F 2 "" H 5200 4600 50  0001 C CNN
+F 3 "" H 5200 4600 50  0001 C CNN
+	1    5200 4600
+	1    0    0    -1
+$EndComp
+Wire Wire Line
+	5200 4400 5200 4600
+$Comp
+L Power_Protection:TPD4E02B04DQA DA6
+U 1 1 637690F2
+P 6550 4400
+F 0 "DA6" V 6133 4450 50  0000 C CNN
+F 1 "TPD4E02B04DQA" V 6224 4450 50  0000 C CNN
+F 2 "Package_SON:USON-10_2.5x1.0mm_P0.5mm" H 6850 4400 50  0001 L CNN
+F 3 "http://www.ti.com/lit/ds/symlink/tpd4e02b04.pdf" H 6675 4725 50  0001 C CNN
+	1    6550 4400
+	0    -1   1    0
+$EndComp
+Wire Wire Line
+	5700 4300 6250 4300
+Wire Wire Line
+	5700 4200 6250 4200
+Wire Wire Line
+	5700 4500 6250 4500
+Wire Wire Line
+	5700 4600 6250 4600
+Wire Wire Line
+	6900 4400 6900 4600
 $EndSCHEMATC

Commit message: U19 changed to upstream KiCAD symbol TFP410PAP
Parts:
- removed U19: TFP410, Package_QFP:HTQFP-64-1EP_10x10mm_P0.5mm_EP8x8mm_Mask4.4x4.4mm_ThermalVias, symbol ecp5_mainboard-rescue:TFP410-pkl_texas
- added U19: TFP410PAP, Package_QFP:HTQFP-64-1EP_10x10mm_P0.5mm_EP8x8mm_Mask4.4x4.4mm_ThermalVias, symbol Video:TFP410PAP
Connections:
- wire segments 630 -> 614
Other:
- moved on the sheet: C123, C124, C125, C126, C127, C128, C129, C130, C131, FB4, FB5, FB6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
