File: hardware/ecp5_mainboard/serdes.sch (KiCad schematic (older format))
At the start: 49 parts, among them J14 9774025151R, J8 9774025151R, P1 M2_SOCKET_E, P3 PCIe_x4_EDGE, U11 CBTL02043A, U15 ECP5UM5G_85_CABGA756, U16 5P49V6965, Y1 25MHz

Commit message: DA1-DA6 changed to upstream symbol TPD4E02B04DQA
Parts:
- removed DA1, DA2, DA3, DA4: TPD4E02B04, Custom Parts:USON10, symbol eco_interface:TPD4E02B04
- added DA1, DA2, DA3, DA4: TPD4E02B04DQA, Package_SON:USON-10_2.5x1.0mm_P0.5mm, symbol Power_Protection:TPD4E02B04DQA
Connections:
- wire segments 384 -> 328

Commit message: U16 changed to upstream KiCAD symbol
Parts:
- removed U16: 5P49V6965, Package_DFN_QFN:QFN-24-1EP_4x4mm_P0.5mm_EP2.7x2.7mm, symbol eco_glue:5P49V6965
- added U16: 5P49V6965, Package_DFN_QFN:QFN-24-1EP_4x4mm_P0.5mm_EP2.8x2.8mm, symbol Oscillator:5P49V6965
Connections:
- wire segments 328 -> 331
Other:
- moved on the sheet: C115, C117, R57, R58, Y1

Commit message: U11 changed to upstream KiCAD symbol CBTL02043A
Parts:
- removed U11: CBTL02043A, Package_DFN_QFN:WQFN-20-1EP_2.5x4.5mm_P0.5mm_EP1x2.9mm, symbol eco_glue:CBTL02043A
- added U11: CBTL02043A, Package_DFN_QFN:WQFN-20-1EP_2.5x4.5mm_P0.5mm_EP1x2.9mm, symbol Analog_Switch:CBTL02043A
Connections:
- wire segments 331 -> 324
Other:
- moved on the sheet: C111, C257, R53, R54
Changed lines of the file:
@@
 Text Label 14800 4050 2    50   ~ 0
 CLKAUXO-
-Text Label 12150 5700 0    50   ~ 0
+Text Label 12350 5700 0    50   ~ 0
 DCU1_REFCLK+
 Wire Wire Line
-	12150 5700 12850 5700
-Text Label 12150 5800 0    50   ~ 0
+	12350 5700 13050 5700
+Text Label 12350 5800 0    50   ~ 0
 DCU1_REFCLK-
 Wire Wire Line
-	12150 5800 12850 5800
+	12350 5800 13050 5800
 $Comp
 L Device:R_Small R47
@@
 	8750 3050 8750 2950
 Connection ~ 8750 2950
-$Comp
-L eco_glue:CBTL02043A U11
-U 1 1 652CFC30
-P 13550 6500
-F 0 "U11" H 13150 7800 50  0000 C CNN
-F 1 "CBTL02043A" H 13900 7800 50  0000 C CNN
-F 2 "Package_DFN_QFN:WQFN-20-1EP_2.5x4.5mm_P0.5mm_EP1x2.9mm" H 13575 6500 50  0001 C CNN
-F 3 "" H 13575 6500 50  0001 C CNN
-	1    13550 6500
-	1    0    0    -1
-$EndComp
-Text Label 12150 6100 0    50   ~ 0
+Text Label 12350 6100 0    50   ~ 0
 M2_REFCLK+
 Wire Wire Line
-	12150 6100 12850 6100
-Text Label 12150 6200 0    50   ~ 0
+	12350 6100 13050 6100
+Text Label 12350 6200 0    50   ~ 0
 M2_REFCLK-
 Wire Wire Line
-	12150 6200 12850 6200
+	12350 6200 13050 6200
 Text Label 14950 5700 2    50   ~ 0
 M2_REFCLK+
@@
 L power:GND #PWR0207
 U 1 1 5C78E250
-P 12700 7250
-F 0 "#PWR0207" H 12700 7000 50  0001 C CNN
-F 1 "GND" H 12705 7077 50  0000 C CNN
-F 2 "" H 12700 7250 50  0001 C CNN
-F 3 "" H 12700 7250 50  0001 C CNN
-	1    12700 7250
-	1    0    0    -1
-$EndComp
-Wire Wire Line
-	12850 6850 12700 6850
-Wire Wire Line
-	12700 6850 12700 6950
-Wire Wire Line
-	12850 6950 12700 6950
-Connection ~ 12700 6950
-Wire Wire Line
-	12700 6950 12700 7050
-Wire Wire Line
-	12700 7050 12850 7050
-Connection ~ 12700 7050
-Wire Wire Line
-	12700 7050 12700 7150
+P 12850 7100
+F 0 "#PWR0207" H 12850 6850 50  0001 C CNN
+F 1 "GND" H 12855 6927 50  0000 C CNN
+F 2 "" H 12850 7100 50  0001 C CNN
+F 3 "" H 12850 7100 50  0001 C CNN
+	1    12850 7100
+	1    0    0    -1
+$EndComp
 $Comp
 L Device:R_Small R54
 U 1 1 5C83C987
-P 12650 6550
-F 0 "R54" V 12454 6550 50  0000 C CNN
-F 1 "10k" V 12545 6550 50  0000 C CNN
-F 2 "Resistor_SMD:R_0402_1005Metric" H 12650 6550 50  0001 C CNN
-F 3 "~" H 12650 6550 50  0001 C CNN
-	1    12650 6550
-	0    1    1    0
-$EndComp
-Wire Wire Line
-	12750 6550 12850 6550
-$Comp
-L power:GND #PWR0254
-U 1 1 5C8603EA
-P 12400 6550
-F 0 "#PWR0254" H 12400 6300 50  0001 C CNN
-F 1 "GND" V 12405 6422 50  0000 R CNN
-F 2 "" H 12400 6550 50  0001 C CNN
-F 3 "" H 12400 6550 50  0001 C CNN
-	1    12400 6550
-	0    1    1    0
-$EndComp
-Wire Wire Line
-	12550 6550 12400 6550
-Text GLabel 12150 6650 0    50   Input ~ 0
+P 12850 6850
+F 0 "R54" H 13000 6900 50  0000 C CNN
+F 1 "10k" H 13000 6800 50  0000 C CNN
+F 2 "Resistor_SMD:R_0402_1005Metric" H 12850 6850 50  0001 C CNN
+F 3 "~" H 12850 6850 50  0001 C CNN
+	1    12850 6850
+	1    0    0    -1
+$EndComp
+Text GLabel 12350 6600 0    50   Input ~ 0
 M2_CLKSEL
-Wire Wire Line
-	12850 6650 12450 6650
 $Comp
 L Device:R_Small R53
 U 1 1 5C8F7D85
-P 12450 6850
-F 0 "R53" H 12391 6804 50  0000 R CNN
-F 1 "10k" H 12391 6895 50  0000 R CNN
-F 2 "Resistor_SMD:R_0402_1005Metric" H 12450 6850 50  0001 C CNN
-F 3 "~" H 12450 6850 50  0001 C CNN
-	1    12450 6850
+P 12550 6850
+F 0 "R53" H 12500 6800 50  0000 R CNN
+F 1 "10k" H 12500 6900 50  0000 R CNN
+F 2 "Resistor_SMD:R_0402_1005Metric" H 12550 6850 50  0001 C CNN
+F 3 "~" H 12550 6850 50  0001 C CNN
+	1    12550 6850
 	-1   0    0    1
 $EndComp
-Wire Wire Line
-	12700 7050 12450 7050
-Wire Wire Line
-	12450 7050 12450 6950
-Wire Wire Line
-	12450 6750 12450 6650
-Connection ~ 12450 6650
-Wire Wire Line
-	12450 6650 12150 6650
 $Comp
 L power:+3V3 #PWR0255
 U 1 1 5C9FA52C
-P 12650 5250
-F 0 "#PWR0255" H 12650 5100 50  0001 C CNN
-F 1 "+3V3" H 12665 5423 50  0000 C CNN
-F 2 "" H 12650 5250 50  0001 C CNN
-F 3 "" H 12650 5250 50  0001 C CNN
-	1    12650 5250
-	1    0    0    -1
-$EndComp
-Wire Wire Line
-	12850 5500 12650 5500
-Wire Wire Line
-	12650 5500 12650 5400
-Connection ~ 12650 5300
+P 13000 5200
+F 0 "#PWR0255" H 13000 5050 50  0001 C CNN
+F 1 "+3V3" H 13015 5373 50  0000 C CNN
+F 2 "" H 13000 5200 50  0001 C CNN
+F 3 "" H 13000 5200 50  0001 C CNN
+	1    13000 5200
+	1    0    0    -1
+$EndComp
+Wire Wire Line
+	12800 5400 12800 5300
 $Comp
 L Device:C_Small C111
 U 1 1 5CA4427D
-P 12450 5300
-F 0 "C111" V 12221 5300 50  0000 C CNN
-F 1 "470n" V 12312 5300 50  0000 C CNN
-F 2 "Capacitor_SMD:C_0402_1005Metric" H 12450 5300 50  0001 C CNN
-F 3 "~" H 12450 5300 50  0001 C CNN
-	1    12450 5300
+P 12600 5200
+F 0 "C111" V 12500 5050 50  0000 C CNN
+F 1 "470n" V 12500 5350 50  0000 C CNN
+F 2 "Capacitor_SMD:C_0402_1005Metric" H 12600 5200 50  0001 C CNN
+F 3 "~" H 12600 5200 50  0001 C CNN
+	1    12600 5200
 	0    1    1    0
 $EndComp
 Wire Wire Line
-	12550 5300 12650 5300
+	12700 5200 12800 5200
 $Comp
 L power:GND #PWR0256
 U 1 1 5CA69A18
-P 11800 5300
-F 0 "#PWR0256" H 11800 5050 50  0001 C CNN
-F 1 "GND" V 11805 5172 50  0000 R CNN
-F 2 "" H 11800 5300 50  0001 C CNN
-F 3 "" H 11800 5300 50  0001 C CNN
-	1    11800 5300
+P 11950 5200
+F 0 "#PWR0256" H 11950 4950 50  0001 C CNN
+F 1 "GND" V 11955 5072 50  0000 R CNN
+F 2 "" H 11950 5200 50  0001 C CNN
+F 3 "" H 11950 5200 50  0001 C CNN
+	1    11950 5200
 	0    1    1    0
 $EndComp
 Wire Wire Line
-	11800 5300 12200 5300
-Wire Wire Line
-	12700 7150 12850 7150
-Connection ~ 12700 7150
-Wire Wire Line
-	12700 7150 12700 7250
-Wire Wire Line
-	12850 5300 12650 5300
-Wire Wire Line
-	12650 5300 12650 5250
+	11950 5200 12350 5200
 $Comp
 L power:GND #PWR0257
@@
 Wire Wire Line
 	8000 10100 8000 10000
-Wire Wire Line
-	12650 5400 12850 5400
-Connection ~ 12650 5400
-Wire Wire Line
-	12650 5400 12650 5300
+Connection ~ 12800 5300
+Wire Wire Line
+	12800 5300 12800 5200
 $Comp
 L Device:C_Small C257
 U 1 1 5C836F58
-P 12450 5500
-F 0 "C257" V 12221 5500 50  0000 C CNN
-F 1 "470n" V 12312 5500 50  0000 C CNN
-F 2 "Capacitor_SMD:C_0402_1005Metric" H 12450 5500 50  0001 C CNN
-F 3 "~" H 12450 5500 50  0001 C CNN
-	1    12450 5500
+P 12600 5400
+F 0 "C257" V 12700 5250 50  0000 C CNN
+F 1 "470n" V 12700 5550 50  0000 C CNN
+F 2 "Capacitor_SMD:C_0402_1005Metric" H 12600 5400 50  0001 C CNN
+F 3 "~" H 12600 5400 50  0001 C CNN
+	1    12600 5400
 	0    1    1    0
 $EndComp
 Wire Wire Line
-	12550 5500 12650 5500
-Connection ~ 12650 5500
-Wire Wire Line
-	12350 5500 12200 5500
-Wire Wire Line
-	12200 5500 12200 5300
-Connection ~ 12200 5300
-Wire Wire Line
-	12200 5300 12350 5300
+	12700 5400 12800 5400
+Wire Wire Line
+	12500 5400 12350 5400
+Wire Wire Line
+	12350 5400 12350 5200
+Connection ~ 12350 5200
+Wire Wire Line
+	12350 5200 12500 5200
 $Comp
 L power:GND #PWR0258
@@
 Wire Wire Line
 	11750 2600 13250 2600
+$Comp
+L Analog_Switch:CBTL02043A U11
+U 1 1 673D84E7
+P 13650 6200
+F 0 "U11" H 13250 7050 50  0000 C CNN
+F 1 "CBTL02043A" H 13950 7050 50  0000 C CNN
+F 2 "Package_DFN_QFN:WQFN-20-1EP_2.5x4.5mm_P0.5mm_EP1x2.9mm" H 13725 5300 50  0001 C CNN
+F 3 "https://www.nxp.com/docs/en/data-sheet/CBTL02043A_CBTL02043B.pdf" H 13775 5850 50  0001 C CNN
+	1    13650 6200
+	1    0    0    -1
+$EndComp
+Wire Wire Line
+	12800 5300 13000 5300
+Wire Wire Line
+	13000 5200 13000 5300
+Connection ~ 13000 5300
+Wire Wire Line
+	13000 5300 13650 5300
+Wire Wire Line
+	12850 6700 12850 6750
+Wire Wire Line
+	12850 6700 13050 6700
+Wire Wire Line
+	12850 6950 12850 7100
+Wire Wire Line
+	12850 7100 13650 7100
+Connection ~ 12850 7100
+Wire Wire Line
+	12850 7100 12550 7100
+Wire Wire Line
+	12550 7100 12550 6950
+Wire Wire Line
+	12350 6600 12550 6600
+Wire Wire Line
+	12550 6750 12550 6600
+Connection ~ 12550 6600
+Wire Wire Line
+	12550 6600 13050 6600
 $EndSCHEMATC
